Commit message: jointTrajectoryController

File: ws/src/pr_description/urdf/pr_robot.xacro (robot description, xacro)
@@ -1,6 +1,12 @@
 <?xml version="1.0" ?>
 <robot name="pr_robot" xmlns:xacro="http://www.ros.org/wiki/xacro">
+<xacro:arg name="use_sim" default="true"/>
 <xacro:include filename="$(find pr_description)/urdf/materials.xacro" />
 <xacro:include filename="$(find pr_description)/urdf/pr_robot.gazebo" />
+<link name="world"/>
+<joint name="world_joint" type="fixed">
+  <parent link="world"/>
+  <child link="base_link"/>
+</joint>
 <link name="base_link">
   <inertial>
@@ -144,5 +150,5 @@
 </link>
 <joint name="yaw_joint" type="revolute">
-  <origin xyz="0.0 0.012 0.036" rpy="0.0 0.0 0.0"/>
+  <origin xyz="0.0 0.012 0.036" rpy="0.0 0.0 3.14159"/>
   <parent link="base_link"/>
   <child link="yaw_link"/>
@@ -154,5 +160,5 @@
   <parent link="yaw_link"/>
   <child link="bicep_link"/>
-  <axis xyz="-1.0 0.0 0.0"/>
+  <axis xyz="1.0 0.0 0.0"/>
   <limit upper="1.570796" lower="0.0" effort="100" velocity="100"/>
 </joint>
@@ -161,5 +167,5 @@
   <parent link="bicep_link"/>
   <child link="forearm_link"/>
-  <axis xyz="-1.0 0.0 0.0"/>
+  <axis xyz="1.0 0.0 0.0"/>
   <limit upper="0.785398" lower="-1.570796" effort="100" velocity="100"/>
 </joint>
@@ -181,4 +187,5 @@
   <child link="pen_tip_link"/>
 </joint>
+<xacro:if value="$(arg use_sim)">
 <ros2_control name="pr_robot" type="system">
   <hardware>
@@ -200,9 +207,38 @@
     <state_interface name="velocity"/>
   </joint>
-  <joint name="pen_mount_joint">
-    <command_interface name="position"/>
-    <state_interface name="position"/>
-    <state_interface name="velocity"/>
-  </joint>
 </ros2_control>
+</xacro:if>
+<xacro:unless value="$(arg use_sim)">
+<ros2_control name="DynamixelHardware" type="system">
+  <hardware>
+    <plugin>dynamixel_hardware/DynamixelHardware</plugin>
+    <param name="usb_port">/dev/ttyUSB0</param>
+    <param name="baud_rate">1000000</param>
+  </hardware>
+  <joint name="forearm_joint">
+    <param name="id">11</param>
+    <param name="profile_acceleration">50</param>
+    <param name="profile_velocity">200</param>
+    <command_interface name="position"/>
+    <state_interface name="position"/>
+    <state_interface name="velocity"/>
+  </joint>
+  <joint name="yaw_joint">
+    <param name="id">12</param>
+    <param name="profile_acceleration">50</param>
+    <param name="profile_velocity">200</param>
+    <command_interface name="position"/>
+    <state_interface name="position"/>
+    <state_interface name="velocity"/>
+  </joint>
+  <joint name="bicep_joint">
+    <param name="id">13</param>
+    <param name="profile_acceleration">50</param>
+    <param name="profile_velocity">200</param>
+    <command_interface name="position"/>
+    <state_interface name="position"/>
+    <state_interface name="velocity"/>
+  </joint>
+</ros2_control>
+</xacro:unless>
 </robot>

Commit message: radi i sim direktna

File: ws/src/pr_description/urdf/pr_robot.xacro (robot description, xacro)
@@ -23,7 +23,7 @@
   </visual>
   <collision>
-    <origin xyz="0 0 0" rpy="0 0 0"/>
-    <geometry>
-      <mesh filename="package://pr_description/meshes/base_link.stl" scale="0.001 0.001 0.001"/>
+    <origin xyz="0.0 0.0 0.0175" rpy="0 0 0"/>
+    <geometry>
+      <box size="0.044 0.080 0.041"/>
     </geometry>
   </collision>
@@ -43,7 +43,7 @@
   </visual>
   <collision>
-    <origin xyz="0 0 0" rpy="0 0 0"/>
-    <geometry>
-      <mesh filename="package://pr_description/meshes/yaw_link.stl" scale="0.001 0.001 0.001"/>
+    <origin xyz="0.0 0.0 0.026" rpy="0 0 0"/>
+    <geometry>
+      <box size="0.056 0.029 0.052"/>
     </geometry>
   </collision>
@@ -63,7 +63,7 @@
   </visual>
   <collision>
-    <origin xyz="0 0 0" rpy="0 0 0"/>
-    <geometry>
-      <mesh filename="package://pr_description/meshes/bicep_link.stl" scale="0.001 0.001 0.001"/>
+    <origin xyz="0.019 0.0 0.091" rpy="0 0 0"/>
+    <geometry>
+      <box size="0.042 0.029 0.188"/>
     </geometry>
   </collision>
@@ -83,7 +83,7 @@
   </visual>
   <collision>
-    <origin xyz="0 0 0" rpy="0 0 0"/>
-    <geometry>
-      <mesh filename="package://pr_description/meshes/forearm_link.stl" scale="0.001 0.001 0.001"/>
+    <origin xyz="0.019 0.078 0.0" rpy="0 0 0"/>
+    <geometry>
+      <box size="0.056 0.167 0.021"/>
     </geometry>
   </collision>
@@ -103,7 +103,7 @@
   </visual>
   <collision>
-    <origin xyz="0 0 0" rpy="0 0 0"/>
-    <geometry>
-      <mesh filename="package://pr_description/meshes/pen_mount_link.stl" scale="0.001 0.001 0.001"/>
+    <origin xyz="0.005 0.029 0.009" rpy="0 0 0"/>
+    <geometry>
+      <box size="0.052 0.066 0.061"/>
     </geometry>
   </collision>
@@ -123,7 +123,7 @@
   </visual>
   <collision>
-    <origin xyz="0 0 0" rpy="0 0 0"/>
-    <geometry>
-      <mesh filename="package://pr_description/meshes/pen_link.stl" scale="0.001 0.001 0.001"/>
+    <origin xyz="0.0 0.0 0.023" rpy="0 0 0"/>
+    <geometry>
+      <cylinder radius="0.006" length="0.132"/>
     </geometry>
   </collision>
@@ -145,5 +145,5 @@
     <origin xyz="0 0 0" rpy="0 0 0"/>
     <geometry>
-      <mesh filename="package://pr_description/meshes/pen_tip_link.stl" scale="0.001 0.001 0.001"/>
+      <sphere radius="0.001"/>
     </geometry>
   </collision>
@@ -203,4 +203,9 @@
   </joint>
   <joint name="forearm_joint">
+    <command_interface name="position"/>
+    <state_interface name="position"/>
+    <state_interface name="velocity"/>
+  </joint>
+  <joint name="pen_mount_joint">
     <command_interface name="position"/>
     <state_interface name="position"/>

Commit message: radi path i pisanje slova

File: ws/src/pr_description/urdf/pr_robot.xacro (robot description, xacro)
@@ -161,5 +161,5 @@
   <child link="bicep_link"/>
   <axis xyz="1.0 0.0 0.0"/>
-  <limit upper="1.570796" lower="0.0" effort="100" velocity="100"/>
+  <limit upper="1.570796" lower="-1.570796" effort="100" velocity="100"/>
 </joint>
 <joint name="forearm_joint" type="revolute">
@@ -168,5 +168,5 @@
   <child link="forearm_link"/>
   <axis xyz="1.0 0.0 0.0"/>
-  <limit upper="0.785398" lower="-1.570796" effort="100" velocity="100"/>
+  <limit upper="1.570796" lower="-1.570796" effort="100" velocity="100"/>
 </joint>
 <joint name="pen_mount_joint" type="revolute">
